File: Seminar_Med_Tech/ECG_Power_Supplies.sch (KiCad schematic (older format))
At the start: 45 parts, among them U1 TPS6, U2 TPS7, U3 TPS7, U4 TPS7

Commit message: add ECG Power Supply
Parts:
- C1, C16, C17, C18, C19, C20, C21, C22, C5, C9: value C -> 10uF
- C10, C11, C12: value C -> NI
- C13, C14, C15, C2: value C -> 2.2uF
- C23: value C -> 0.1uF
- C3, C4, C6, C7, C8: value C -> 1uF
- JP2: renamed from JP1; value Jumper_NC_Dual -> JP2
- JP20: renamed from JP2; value Jumper_NC_Dual -> JP20
- L2, L3, L4, L5: value L -> 3.3uH
- R1, R4: value R -> NI
- R2: value R -> 49.9K
- R3: value R -> 47.5K
- R5: value R -> 46.4K
- R6: value R -> 43.2K
Connections:
- wire segments 85 -> 125
Other:
- moved on the sheet: C12, C15, C18, C2, C22, JP20, R3, R6, TP6
