File: Seminar_Med_Tech/Connectors.sch (KiCad schematic (older format))
At the start: 12 parts

Commit message: Changed labels
Changed lines of the file:
@@
 EESchema Schematic File Version 2
+LIBS:Seminar_Med_Tech-rescue
 LIBS:power
 LIBS:device
@@
 LIBS:contrib
 LIBS:valves
-LIBS:ECG_Power_Supplies-cache
 LIBS:MechTech
+LIBS:MedTech
 LIBS:MedTec2
-LIBS:MedTech
-LIBS:Seminar_Med_Tech 4-cache
 LIBS:Seminar_Med_Tech-cache
-LIBS:Seminar_Med_Tech-rescue
-LIBS:Connectors-cache
 EELAYER 25 0
 EELAYER END
 $Descr A4 11693 8268
 encoding utf-8
-Sheet 1 1
+Sheet 2 3
 Title ""
 Date ""
@@
 	2325 4250 2550 4250
 Wire Wire Line
-	7325 5750 7600 5750
-Wire Wire Line
-	7600 5750 7675 5750
+	7325 5750 7675 5750
 Wire Wire Line
 	7600 5525 7600 5750
@@
 	9850 5500 9850 5775
 Wire Wire Line
-	1350 3550 1525 3550
-Wire Wire Line
-	1525 3550 2550 3550
-Wire Wire Line
-	1525 2600 1525 2700
-Wire Wire Line
-	1525 2700 1525 3550
+	1350 3550 2550 3550
+Wire Wire Line
+	1525 2600 1525 3550
 Connection ~ 1525 3550
 Wire Wire Line
-	1525 2700 1725 2700
-Wire Wire Line
-	1725 2700 1850 2700
+	1525 2700 1850 2700
 Connection ~ 1525 2700
 Wire Wire Line
@@
 	2150 2700 2275 2700
 Wire Wire Line
-	2275 2700 2275 2850
-Wire Wire Line
-	2275 2850 2275 2975
+	2275 2700 2275 2975
 Wire Wire Line
 	2275 2975 2150 2975
@@
 	3050 3550 3550 3550
 Wire Wire Line
-	4150 3550 4500 3550
-Wire Wire Line
-	4500 3550 4875 3550
-Wire Wire Line
-	4875 3450 4875 3550
-Wire Wire Line
-	4875 3550 4875 3750
+	4150 3550 4875 3550
+Wire Wire Line
+	4875 3450 4875 3750
 Wire Wire Line
 	4500 3750 4500 3550
