File: Seminar_Med_Tech/Connectors.sch (KiCad schematic (older format))
At the start: 13 parts, among them J2 CONN_01X10, J3 CONN_02X10, J5 CONN_02X10

Commit message: jumper
Parts:
- C68, C69, C70, C71: footprint (none) -> Capacitors_SMD:C_1206_HandSoldering
- J2: footprint (none) -> Pin_Headers:Pin_Header_Straight_1x10_Pitch2.54mm
- J3, J5: footprint (none) -> Pin_Headers:Pin_Header_Straight_2x10_Pitch2.54mm
- JP21: footprint (none) -> jumper:jumper1x3
- JP3: footprint (none) -> jumper:Jumper1x2
- R67, R74: footprint (none) -> Resistors_SMD:R_0805_HandSoldering
- TP10, TP7: footprint (none) -> Measurement_Points:Test_Point_Keystone_5000-5004_Miniature
Changed lines of the file:
@@
 F 0 "J3" H 2800 4550 50  0000 C CNN
 F 1 "CONN_02X10" V 2800 4000 50  0000 C CNN
-F 2 "" H 2800 2800 50  0001 C CNN
+F 2 "Pin_Headers:Pin_Header_Straight_2x10_Pitch2.54mm" H 2800 2800 50  0001 C CNN
 F 3 "" H 2800 2800 50  0001 C CNN
 	1    2800 4000
@@
 F 0 "J5" H 7600 4525 50  0000 C CNN
 F 1 "CONN_02X10" V 7600 3975 50  0000 C CNN
-F 2 "" H 7600 2775 50  0001 C CNN
+F 2 "Pin_Headers:Pin_Header_Straight_2x10_Pitch2.54mm" H 7600 2775 50  0001 C CNN
 F 3 "" H 7600 2775 50  0001 C CNN
 	1    7600 3975
@@
 F 0 "JP21" H 7275 5650 50  0000 L CNN
 F 1 "Jumper_NC_Dual" H 7225 5850 50  0000 C BNN
-F 2 "" H 7225 5750 50  0001 C CNN
+F 2 "jumper:jumper1x3" H 7225 5750 50  0001 C CNN
 F 3 "" H 7225 5750 50  0001 C CNN
 	1    7225 5750
@@
 F 0 "R67" V 7680 5375 50  0000 C CNN
 F 1 "10K" V 7600 5375 50  0000 C CNN
-F 2 "" V 7530 5375 50  0001 C CNN
+F 2 "Resistors_SMD:R_0805_HandSoldering" V 7530 5375 50  0001 C CNN
 F 3 "" H 7600 5375 50  0001 C CNN
 	1    7600 5375
@@
 $EndComp
 $Comp
-L GND #PWR03
+L GND #PWR01
 U 1 1 593AE084
 P 7225 6000
-F 0 "#PWR03" H 7225 5750 50  0001 C CNN
+F 0 "#PWR01" H 7225 5750 50  0001 C CNN
 F 1 "GND" H 7225 5850 50  0000 C CNN
 F 2 "" H 7225 6000 50  0001 C CNN
@@
 $EndComp
 $Comp
-L GND #PWR04
+L GND #PWR02
 U 1 1 593AE114
 P 3675 5000
-F 0 "#PWR04" H 3675 4750 50  0001 C CNN
+F 0 "#PWR02" H 3675 4750 50  0001 C CNN
 F 1 "GND" H 3675 4850 50  0000 C CNN
 F 2 "" H 3675 5000 50  0001 C CNN
@@
 $EndComp
 $Comp
-L GND #PWR05
+L GND #PWR03
 U 1 1 593AE149
 P 9375 3700
-F 0 "#PWR05" H 9375 3450 50  0001 C CNN
+F 0 "#PWR03" H 9375 3450 50  0001 C CNN
 F 1 "GND" H 9375 3550 50  0000 C CNN
 F 2 "" H 9375 3700 50  0001 C CNN
@@
 SPI_CS1
 $Comp
-L GND #PWR06
+L GND #PWR04
 U 1 1 593E72B3
 P 9200 5600
-F 0 "#PWR06" H 9200 5350 50  0001 C CNN
+F 0 "#PWR04" H 9200 5350 50  0001 C CNN
 F 1 "GND" H 9200 5450 50  0000 C CNN
 F 2 "" H 9200 5600 50  0001 C CNN
@@
 F 0 "R74" V 9605 5500 50  0000 C CNN
 F 1 "0" V 9525 5500 50  0000 C CNN
-F 2 "" V 9455 5500 50  0001 C CNN
+F 2 "Resistors_SMD:R_0805_HandSoldering" V 9455 5500 50  0001 C CNN
 F 3 "" H 9525 5500 50  0001 C CNN
 	1    9525 5500
@@
 F 0 "TP10" H 1350 3820 50  0000 C CNN
 F 1 "TEST" H 1350 3750 50  0000 C CNN
-F 2 "" H 1550 3550 50  0001 C CNN
+F 2 "Measurement_Points:Test_Point_Keystone_5000-5004_Miniature" H 1550 3550 50  0001 C CNN
 F 3 "" H 1550 3550 50  0001 C CNN
 	1    1350 3550
@@
 F 0 "C71" H 2025 2800 50  0000 L CNN
 F 1 "100uF" H 2025 2600 50  0000 L CNN
-F 2 "" H 2038 2550 50  0001 C CNN
+F 2 "Capacitors_SMD:C_1206_HandSoldering" H 2038 2550 50  0001 C CNN
 F 3 "" H 2000 2700 50  0001 C CNN
 	1    2000 2700
@@
 F 0 "C70" H 2025 3075 50  0000 L CNN
 F 1 "0.1uF" H 2025 2875 50  0000 L CNN
-F 2 "" H 2038 2825 50  0001 C CNN
+F 2 "Capacitors_SMD:C_1206_HandSoldering" H 2038 2825 50  0001 C CNN
 F 3 "" H 2000 2975 50  0001 C CNN
 	1    2000 2975
@@
 F 0 "JP3" H 3850 3700 50  0000 C CNN
 F 1 "Jumper" H 3850 3470 50  0000 C CNN
-F 2 "" H 3850 3550 50  0001 C CNN
+F 2 "jumper:Jumper1x2" H 3850 3550 50  0001 C CNN
 F 3 "" H 3850 3550 50  0001 C CNN
 	1    3850 3550
@@
 F 0 "TP7" H 4275 3820 50  0000 C CNN
 F 1 "TEST" H 4275 3750 50  0000 C CNN
-F 2 "" H 4475 3550 50  0001 C CNN
+F 2 "Measurement_Points:Test_Point_Keystone_5000-5004_Miniature" H 4475 3550 50  0001 C CNN
 F 3 "" H 4475 3550 50  0001 C CNN
 	1    4275 3550
@@
 F 0 "C69" H 4525 4000 50  0000 L CNN
 F 1 "0.1uF" H 4525 3800 50  0000 L CNN
-F 2 "" H 4538 3750 50  0001 C CNN
+F 2 "Capacitors_SMD:C_1206_HandSoldering" H 4538 3750 50  0001 C CNN
 F 3 "" H 4500 3900 50  0001 C CNN
 	1    4500 3900
@@
 F 0 "C68" H 4900 4000 50  0000 L CNN
 F 1 "100uF" H 4900 3800 50  0000 L CNN
-F 2 "" H 4913 3750 50  0001 C CNN
+F 2 "Capacitors_SMD:C_1206_HandSoldering" H 4913 3750 50  0001 C CNN
 F 3 "" H 4875 3900 50  0001 C CNN
 	1    4875 3900
@@
 $EndComp
 $Comp
-L GND #PWR07
+L GND #PWR05
 U 1 1 593E9316
 P 4700 4150
-F 0 "#PWR07" H 4700 3900 50  0001 C CNN
+F 0 "#PWR05" H 4700 3900 50  0001 C CNN
 F 1 "GND" H 4700 4000 50  0000 C CNN
 F 2 "" H 4700 4150 50  0001 C CNN
@@
 F 0 "J2" H 4200 6975 50  0000 C CNN
 F 1 "CONN_01X10" V 4300 6425 50  0000 C CNN
-F 2 "" H 4200 6425 50  0001 C CNN
+F 2 "Pin_Headers:Pin_Header_Straight_1x10_Pitch2.54mm" H 4200 6425 50  0001 C CNN
 F 3 "" H 4200 6425 50  0001 C CNN
 	1    4200 6425
