File: Seminar_Med_Tech/Seminar_Med_Tech 4.sch (KiCad schematic (older format))
At the start: 74 parts, among them J1 CONN_02X08, J7 CONN_02X08, U1 OPA132, U18 ADS1298, U20 ADS1298

Commit message: added footprints
Parts:
- U1: footprint jumper:OSC132 -> (none)
Changed lines of the file:
@@
 F 0 "U1" H 10050 950 60  0000 C CNN
 F 1 "OPA132" H 10025 1300 60  0000 C CNN
-F 2 "jumper:OSC132" H 9925 1100 60  0001 C CNN
+F 2 "" H 9925 1100 60  0001 C CNN
 F 3 "" H 9925 1100 60  0001 C CNN
 	1    9925 1100
