File: Seminar_Med_Tech/Seminar_Med_Tech.kicad_pcb (KiCad board)
At the start: 2 copper layers, 165 parts, among them J1 CONN_02X08, J2 CONN_02X08, J3 CONN_02X10, J5 CONN_02X10, J6 DB15_F-RA, J7 CONN_02X08, U1 OPA132, U18 ADS1298, U20 ADS1298, U4 LM317T, U5 LM317T, U6 LM337K

Commit message: Update
Parts:
- removed J2: CONN_02X08, Pin_Headers:Pin_Header_Straight_2x08_Pitch2.54mm
- added PSK5: CONN_02X08, Pin_Headers:Pin_Header_Straight_2x08_Pitch2.54mm, F.Cu at (114.3, 67.3)
- moved TP8 194.6 mm to (338.9, 65.0)
- moved R67 191.6 mm to (337.0, 70.7)
- moved JP21 191.2 mm to (333.8, 58.1)
- moved TP7 190.9 mm to (335.2, 65.0)
- moved JP2 186.1 mm to (330.4, 65.5)
- moved C68 185.5 mm to (331.0, 71.8)
- moved R74 180.7 mm to (327.1, 77.6)
- moved C69 174.8 mm to (321.1, 77.5)
- moved C33 167.9 mm to (314.1, 77.5)
- moved PSK1 162.0 mm to (292.9, 57.9)
- moved C27 161.0 mm to (307.2, 77.5)
- moved PSK2 156.5 mm to (27.9, 25.4)
- moved JP3 154.6 mm to (300.8, 78.2)
- moved TP1 139.3 mm to (279.4, 57.6)
- moved R11 138.2 mm to (280.3, 63.3)
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Connections:
- J1 pad 1: ECG_16N -> ECG_13P
- J1 pad 11: ECG_14P -> ECG_15N
- J1 pad 13: ECG_13N -> ECG_16P
- J1 pad 15: ECG_13P -> ECG_16N
- J1 pad 3: ECG_16P -> ECG_13N
- J1 pad 5: ECG_15N -> ECG_14P
- J1 pad 7: ECG_15P -> ECG_14N
- J1 pad 9: ECG_14N -> ECG_15P
Routing:
- net ECG_4P: track 0.00 -> 74.2 mm
- net ECG_3P: track 0.00 -> 69.9 mm
- net ECG_2P: track 0.00 -> 65.7 mm
- net ECG_4N: track 0.00 -> 65.7 mm
- net ECG_3N: track 0.00 -> 63.3 mm
- net ECG_5P: track 0.00 -> 61.6 mm
- net ECG_1P: track 0.00 -> 61.5 mm
- net ECG_6P: track 0.00 -> 61.4 mm
- net ECG_7P: track 0.00 -> 59.4 mm
- net ECG_2N: track 0.00 -> 59.0 mm
- net ECG_5N: track 0.00 -> 56.3 mm
- net ECG_1N: track 0.00 -> 54.8 mm
- net ECG_6N: track 0.00 -> 54.3 mm
- net ECG_8P: track 0.00 -> 54.0 mm
- net ECG_8N: track 0.00 -> 53.0 mm
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
Commit message: Update
Parts:
- added C34: 1uF, Capacitors_SMD:C_1206_HandSoldering, F.Cu at (137.8, 96.5)
- added C35: 0.1uF, Capacitors_SMD:C_1206_HandSoldering, F.Cu at (137.8, 100.3)
- C45, C46: footprint Capacitors_SMD:CP_Elec_4x5.8 -> Jumper:4mmx5,5mmSMDElec
- C47, C48: footprint Capacitors_SMD:CP_Elec_4x5.8 -> Jumper:4mmx5,5mmSMDElec10uf
- moved TP8 169.7 mm to (175.0, 108.7)
- moved R4 163.7 mm to (113.0, 23.5)
- moved TP7 162.8 mm to (174.2, 89.4)
- moved TP1 162.4 mm to (118.7, 81.3)
- moved C21 157.9 mm to (92.1, 24.8)
- moved JP2 156.5 mm to (178.8, 104.4), turned to 270 degrees
- moved C68 151.3 mm to (180.7, 89.5)
- moved R8 148.4 mm to (123.8, 39.4), turned to 90 degrees
- moved R11 145.3 mm to (143.5, 112.4), turned to 270 degrees
- moved R67 144.7 mm to (192.5, 78.7), turned to 270 degrees
- moved C95 143.7 mm to (126.4, 80.0), turned to 90 degrees
- moved R1 142.4 mm to (138.4, 23.5), turned to 270 degrees
- moved C69 140.7 mm to (180.6, 85.1)
- moved C8 139.9 mm to (133.3, 123.8), turned to 90 degrees
- moved C22 138.1 mm to (108.0, 17.1), turned to 270 degrees
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Connections:
- C27 pad 1: VCC_3.3V -> 3.3V_Supply
- C33 pad 1: VCC_3.3V -> 3.3V_Supply
- C68 pad 1: VCC_5V -> 5V_Supply
- C69 pad 1: VCC_5V -> 5V_Supply
- J3 pad 15: EXT_CLK -> SPI_CS2
- J5 pad 16: Net-(J5-Pad16) -> GPIO14
- J5 pad 18: Net-(J5-Pad18) -> GPIO24
- J5 pad 20: SPI_CS2 -> EXT_CLK
- J7 pad 1: PACEOUT21 -> PACEOUT22
- J7 pad 10: GPIO23 -> GPIO11
- J7 pad 11: GPIO11 -> Net-(J7-Pad11)
- J7 pad 12: Net-(J7-Pad12) -> GPIO12
- J7 pad 13: GPIO12 -> Net-(J7-Pad13)
- J7 pad 14: DAISY_IN -> GPIO13
- J7 pad 15: GPIO21 -> DAISY_IN
- J7 pad 2: PACEOUT22 -> PACEOUT11
- J7 pad 3: PACEOUT11 -> PACEOUT21
- J7 pad 5: GPIO13 -> GPIO23
- J7 pad 6: GPIO22 -> /PWDN
- J7 pad 7: GPIO14 -> GPIO22
- J7 pad 8: /PWDN -> Net-(J7-Pad8)
- J7 pad 9: GPIO24 -> GPIO21
- JP2 pad 2: VCC_3.3V -> 3.3V_Supply
- JP3 pad 2: VCC_5V -> 5V_Supply
- TP7 pad 1: VCC_5V -> 5V_Supply
- TP8 pad 1: VCC_3.3V -> 3.3V_Supply
- U18 pad 55: Net-(C13-Pad2) -> Net-(C34-Pad2)
Routing:
- net ECG_5P: track 61.6 -> 13.8 mm
- net AVDD: track 0.00 -> 42.6 mm
- net ECG_5N: track 56.3 -> 19.0 mm
- net Net-(JP30-Pad2): track 20.9 -> 0.00 mm
- net Net-(JP30-Pad4): track 20.3 -> 0.00 mm
- net ECG_6P: track 61.4 -> 41.8 mm
- net Net-(JP31-Pad2): track 16.5 -> 0.00 mm
- net ECG_6N: track 54.3 -> 41.6 mm
- net ECG_4N: track 65.7 -> 58.8 mm
- net ECG_4P: track 74.2 -> 67.3 mm
- net ECG_3N: track 63.3 -> 57.6 mm
- net ECG_3P: track 69.9 -> 65.0 mm
- net /ADC1298_ECG_FE/ELEC_RA: track 28.6 -> 24.6 mm
- net ECG_V1: track 7.76 -> 3.88 mm
- net /ADC1298_ECG_FE/ELEC_V2: track 37.8 -> 34.0 mm
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
Commit message: Update
Parts:
- moved J5 20.2 mm to (177.5, 51.6)
- moved C14 12.7 mm to (226.7, 138.3)
- moved C18 12.7 mm to (226.7, 119.9)
- moved C39 12.7 mm to (230.1, 78.5)
- moved C4 12.7 mm to (226.7, 129.4)
- moved C42 12.7 mm to (227.1, 65.8)
- moved C47 12.7 mm to (227.1, 39.6)
- moved C48 12.7 mm to (233.2, 99.3)
- moved C6 12.7 mm to (226.7, 133.9)
- moved D13 12.7 mm to (235.7, 76.7)
- moved PSK3 12.7 mm to (250.4, 68.1)
- moved R20 12.7 mm to (227.1, 69.8)
- moved R27 12.7 mm to (232.4, 73.7)
- moved R32 12.7 mm to (232.4, 48.0)
- moved R35 12.7 mm to (233.4, 94.5)
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Connections:
- J5 pad 11: I/O_2 -> I/O_5
- J5 pad 13: I/O_3 -> I/O_6
- J5 pad 15: I/O_4 -> I/O_7
- J5 pad 17: I/O_5 -> I/O_8
- J5 pad 4: I/O_6 -> I/O_1
- J5 pad 6: I/O_7 -> I/O_2
- J5 pad 8: I/O_8 -> I/O_3
- J5 pad 9: I/O_1 -> I/O_4
Routing:
- net ECG_5P: track 13.8 -> 51.5 mm
- net ECG_5N: track 19.0 -> 47.1 mm
- net ECG_6P: track 41.8 -> 51.9 mm
- net ECG_8P: track 54.0 -> 45.4 mm
- net ECG_8N: track 53.0 -> 46.1 mm
- net ECG_7N: track 49.3 -> 42.9 mm
- net ECG_4N: track 58.8 -> 52.5 mm
- net ECG_2P: track 62.7 -> 56.3 mm
- net ECG_2N: track 56.0 -> 49.6 mm
- net ECG_4P: track 67.3 -> 61.1 mm
- net ECG_1N: track 53.7 -> 47.6 mm
- net ECG_1P: track 60.3 -> 54.2 mm
- net ECG_3P: track 65.0 -> 58.9 mm
- net ECG_7P: track 56.7 -> 50.7 mm
- net ECG_3N: track 57.6 -> 52.0 mm
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
Commit message: Update
Parts:
- moved PSK2 63.2 mm to (17.0, 86.2), turned to 180 degrees
- moved JP15 57.6 mm to (97.0, 42.7), turned to 0 degrees
- moved JP21 46.9 mm to (220.3, 36.0), turned to 180 degrees
- moved R67 42.7 mm to (190.9, 36.1), turned to 180 degrees
- moved R1 33.7 mm to (132.7, 56.7), turned to 180 degrees
- moved JP37 31.1 mm to (94.5, 111.7), turned to 270 degrees
- moved R5 30.6 mm to (127.6, 56.7)
- moved C21 29.2 mm to (114.0, 44.1)
- moved JP36 21.9 mm to (101.3, 111.7), turned to 270 degrees
- moved U1 20.3 mm to (116.0, 41.9)
- moved C22 19.0 mm to (114.2, 35.1), turned to 0 degrees
- moved R2 18.8 mm to (132.9, 52.3)
- moved C34 17.9 mm to (150.6, 95.8)
- moved C35 17.9 mm to (150.6, 99.6)
- moved JP30 16.8 mm to (94.4, 99.1), turned to 90 degrees
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Routing:
- net Net-(JP37-Pad4): track 0.00 -> 143.9 mm
- net AVDD: track 41.4 -> 180.8 mm, vias 0 -> 12
- net Net-(JP37-Pad2): track 0.00 -> 137.9 mm
- net Net-(JP36-Pad4): track 0.00 -> 129.9 mm
- net Net-(JP36-Pad2): track 0.00 -> 118.0 mm
- net SPI_START: track 0.00 -> 110.9 mm, vias 0 -> 2
- net CLKSEL: track 0.00 -> 105.5 mm
- net /ADC1298_ECG_FE/ELEC_SHD: track 0.00 -> 104.9 mm, vias 0 -> 4
- net Net-(JP35-Pad4): track 0.00 -> 100.3 mm
- net Net-(JP35-Pad2): track 0.00 -> 87.9 mm
- net /ADC1298_ECG_FE/ELEC_V4: track 36.6 -> 119.7 mm, vias 1 -> 4
- net Net-(C20-Pad1): track 0.00 -> 82.8 mm
- net /ADC1298_ECG_FE/ELEC_V5: track 22.1 -> 104.0 mm, vias 1 -> 2
- net /ADC1298_ECG_FE/ELEC_RL: track 0.00 -> 74.9 mm, vias 0 -> 2
- net AGND: track 0.00 -> 73.6 mm, vias 0 -> 32
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
Commit message: Update
Parts:
- moved J3 0.57 mm to (178.1, 101.1)
Changed lines of the file:
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@@
   )
   (module Pin_Headers:Pin_Header_Straight_2x10_Pitch2.54mm (layer F.Cu)
-    (at 177.546 101.346 90)
+    (at 178.054 101.092 90)
     (descr "Through hole straight pin header, 2x10, 2.54mm pitch, double rows")
     (tags "Through hole pin header THT 2x10 2.54mm double row")
@@
       (effects (font (size 1 1) (thickness 0.15)))
     )
-    (fp_text value CONN_02X10 (at 1.27 25.19 90) (layer F.Fab)
+    (fp_text value CONN_02X10 (at 1.27 25.4 90) (layer F.Fab)
       (effects (font (size 1 1) (thickness 0.15)))
     )

Commit message: Update
Parts:
- moved D15 129.5 mm to (108.4, 103.4)
- moved U6 128.3 mm to (107.6, 103.6)
- moved C48 127.9 mm to (105.7, 109.4)
- moved C46 126.9 mm to (100.5, 100.9)
- moved R31 126.9 mm to (102.0, 103.9)
- moved R20 123.6 mm to (104.1, 81.7)
- moved PSK3 120.3 mm to (130.7, 79.2)
- moved C38 118.9 mm to (107.2, 75.9)
- moved C39 118.9 mm to (111.3, 80.5)
- moved R27 118.9 mm to (113.5, 75.7)
- moved D13 118.9 mm to (116.8, 78.7)
- moved U4 118.9 mm to (115.3, 68.8)
- moved C44 114.0 mm to (113.5, 100.7)
- moved R35 114.0 mm to (119.6, 100.7)
- moved TP6 113.4 mm to (104.3, 118.4)
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Routing:
- net AVDD: track 180.8 -> 0.00 mm, vias 12 -> 0
- net Net-(JP37-Pad4): track 143.9 -> 0.00 mm
- net Net-(JP37-Pad2): track 137.9 -> 0.00 mm
- net Net-(JP36-Pad4): track 129.9 -> 0.00 mm
- net /ADC1298_ECG_FE/ELEC_V4: track 119.7 -> 0.00 mm, vias 4 -> 0
- net Net-(JP36-Pad2): track 118.0 -> 0.00 mm
- net SPI_START: track 110.9 -> 0.00 mm, vias 2 -> 0
- net CLKSEL: track 105.5 -> 0.00 mm
- net /ADC1298_ECG_FE/ELEC_SHD: track 104.9 -> 0.00 mm, vias 4 -> 0
- net /ADC1298_ECG_FE/ELEC_V5: track 104.0 -> 0.00 mm, vias 2 -> 0
- net Net-(JP35-Pad4): track 100.3 -> 0.00 mm
- net Net-(JP35-Pad2): track 87.9 -> 0.00 mm
- net /ADC1298_ECG_FE/ELEC_RA: track 83.6 -> 0.00 mm, vias 1 -> 0
- net Net-(C20-Pad1): track 82.8 -> 0.00 mm
- net /ADC1298_ECG_FE/ELEC_V3: track 76.1 -> 0.00 mm, vias 1 -> 0
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Other:
- board outline added: 335.7 x 108.1 mm

Commit message: Update
Parts:
- C11, C12, C14, C16, C17, C18, C20, C21, C23, C24, C26, C28, C29, C30, C31, C32, C4, C5, C6, C72, C73, C74, C75, C76, C77, C80, C82, C84, C86, C88, C91, C92, C93, JP18, JP19, OSC1, R3, R4, R67, R8: moved to B.Cu
- JP16: value Jumper -> Jumper_NC_Dual; footprint Jumper:Jumper1x2 -> Jumper:jumper1x3
- moved R75 78.8 mm to (56.1, 126.0)
- moved C12 53.5 mm to (131.8, 51.7), turned to 180 degrees
- moved C48 53.4 mm to (143.4, 71.7), turned to 180 degrees
- moved C14 53.3 mm to (134.0, 60.6), turned to 90 degrees
- moved C6 51.3 mm to (143.1, 60.5), turned to 90 degrees
- moved R31 49.9 mm to (143.6, 76.4), turned to 0 degrees
- moved C17 49.7 mm to (135.8, 67.2)
- moved R20 48.7 mm to (143.4, 52.9)
- moved C5 48.7 mm to (132.0, 48.7), turned to 180 degrees
- moved R10 48.6 mm to (76.2, 47.8)
- moved R9 48.4 mm to (71.2, 47.9), turned to 180 degrees
- moved C91 48.4 mm to (70.3, 48.0), turned to 180 degrees
- moved D1 48.3 mm to (80.7, 47.8), turned to 180 degrees
- moved C46 47.9 mm to (139.5, 73.2), turned to 180 degrees
- moved C4 47.5 mm to (137.2, 60.6), turned to 90 degrees
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Connections:
- C90 pad 2: Net-(C90-Pad2) -> /WCT
- J1 pad 10: ECG_10N -> ECG_11P
- J1 pad 12: ECG_10P -> ECG_11N
- J1 pad 14: ECG_9N -> ECG_12P
- J1 pad 16: ECG_9P -> ECG_12N
- J1 pad 2: ECG_12N -> ECG_9P
- J1 pad 4: ECG_12P -> ECG_9N
- J1 pad 6: ECG_11N -> ECG_10P
- J1 pad 8: ECG_11P -> ECG_10N
- JP16 pad 2: Net-(C90-Pad2) -> Net-(JP16-Pad2)
- JP22 pad 1: /WCT -> Net-(JP16-Pad2)
- JP23 pad 1: /WCT -> Net-(JP16-Pad2)
- JP24 pad 1: /WCT -> Net-(JP16-Pad2)
- JP25 pad 1: /WCT -> Net-(JP16-Pad2)
- JP26 pad 1: /WCT -> Net-(JP16-Pad2)
- JP29 pad 1: /WCT -> Net-(JP16-Pad2)
- PSK2 pad 10: /ADC1298_ECG_FE/ELEC_RL -> /ADC1298_ECG_FE/ELEC_RA
- PSK2 pad 6: /ADC1298_ECG_FE/ELEC_RA -> /ADC1298_ECG_FE/ELEC_RL
- PSK2 pad 7: /ADC1298_ECG_FE/ELEC_LA -> /ADC1298_ECG_FE/ELEC_V1
- PSK2 pad 9: /ADC1298_ECG_FE/ELEC_V1 -> /ADC1298_ECG_FE/ELEC_LA
- PSK5 pad 10: ECG_2N -> ECG_3P
- PSK5 pad 12: ECG_2P -> ECG_3N
- PSK5 pad 14: ECG_1N -> ECG_4P
- PSK5 pad 16: ECG_1P -> ECG_4N
- PSK5 pad 2: ECG_4N -> ECG_1P
- PSK5 pad 4: ECG_4P -> ECG_1N
- PSK5 pad 6: ECG_3N -> ECG_2P
- PSK5 pad 8: ECG_3P -> ECG_2N
- U20 pad 64: Net-(C90-Pad2) -> /WCT
Routing:
- net AVDD: track 0.00 -> 178.2 mm, vias 0 -> 8
- net DVDD: track 0.00 -> 125.2 mm, vias 0 -> 8
- net /RESET: track 0.00 -> 104.2 mm, vias 0 -> 2
- net AVSS: track 0.00 -> 95.0 mm, vias 0 -> 1
- net /PWDN: track 0.00 -> 84.6 mm, vias 0 -> 7
- net SPI_START: track 0.00 -> 79.8 mm, vias 0 -> 2
- net GPIO24: track 0.00 -> 77.7 mm, vias 0 -> 3
- net /ADC1298_ECG_FE/ELEC_RL: track 0.00 -> 71.4 mm
- net /ADC1298_ECG_FE/ELEC_V1: track 0.00 -> 68.6 mm
- net EXT_CLK: track 0.00 -> 68.3 mm
- net /ADC1298_ECG_FE/ELEC_SHD: track 0.00 -> 65.8 mm
- net /ADC1298_ECG_FE/ELEC_LL: track 0.00 -> 65.2 mm, vias 0 -> 2
- net Net-(JP16-Pad2): track 0.00 -> 63.4 mm, vias 0 -> 1
- net /ADC1298_ECG_FE/ELEC_LA: track 0.00 -> 62.5 mm, vias 0 -> 3
- net /CLK: track 0.00 -> 61.0 mm, vias 0 -> 3
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Other:
- board size 335.7 x 108.1 mm -> 98.6 x 88 mm
