File: Seminar_Med_Tech/Seminar_Med_Tech.kicad_pcb (KiCad board)
At the start: 2 copper layers, 98.6 x 88 mm, 167 parts, among them J1 CONN_02X08, J3 CONN_02X10, J5 CONN_02X10, J6 DB15_F-RA, J7 CONN_02X08, U1 OPA132, U18 ADS1298, U20 ADS1298, U4 LM317T, U5 LM317T, U6 LM337K

Commit message: added connections
Parts:
- C34, C35, C68, C69, R75: moved to B.Cu
- moved R75 90.0 mm to (114.6, 57.6), turned to 270 degrees
- moved TP7 72.6 mm to (118.6, 107.2)
- moved JP3 68.0 mm to (110.6, 100.0), turned to 270 degrees
- moved TP4 66.6 mm to (125.9, 107.2)
- moved TP8 66.4 mm to (137.2, 107.3)
- moved TP5 66.3 mm to (129.5, 107.3)
- moved TP6 66.2 mm to (133.2, 107.3)
- moved TP3 66.1 mm to (122.0, 107.3)
- moved C68 63.9 mm to (129.8, 55.0), turned to 180 degrees
- moved C69 63.5 mm to (124.4, 52.6), turned to 270 degrees
- moved C34 44.1 mm to (95.8, 83.4), turned to 90 degrees
- moved C35 43.6 mm to (98.6, 83.4), turned to 90 degrees
- moved R6 41.8 mm to (112.2, 85.6), turned to 180 degrees
- moved R7 31.5 mm to (104.8, 90.0), turned to 180 degrees
- moved R11 31.1 mm to (107.7, 88.1), turned to 0 degrees
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Routing:
- net 5V_Supply: track 13.2 -> 55.9 mm, vias 0 -> 2
- net AGND: track 14.8 -> 48.7 mm, vias 4 -> 5
- net 3.3V_Supply: track 18.5 -> 52.1 mm
- net Net-(J3-Pad2): track 0.00 -> 23.1 mm
- net DVDD: track 125.2 -> 145.6 mm, vias 8 -> 10
- net Net-(C34-Pad2): track 0.00 -> 15.7 mm, vias 0 -> 1
- net /PWDN: track 84.6 -> 93.0 mm
- net SPI_CS1: track 0.00 -> 6.74 mm, vias 0 -> 1
- net /RESET: track 104.2 -> 109.3 mm
- net AVSS: track 95.0 -> 98.8 mm, vias 1 -> 2
- net Net-(C68-Pad2): track 0.00 -> 3.57 mm
- net GPIO24: track 77.7 -> 81.1 mm
- net GND: track 48.4 -> 50.8 mm
- net GPIO12: track 45.8 -> 47.3 mm
- net GPIO11: track 50.4 -> 51.7 mm
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- added copper zone on B.Cu, net AGND
- added copper zone on F.Cu, net AVSS
Other:
- board size 98.6 x 88 mm -> 96 x 88 mm

Commit message: Update
Parts:
- R12: moved to B.Cu
- moved R6 26.8 mm to (123.3, 61.2), turned to 90 degrees
- moved R12 24.3 mm to (128.1, 67.9), turned to 90 degrees
- moved TP7 7.71 mm to (113.7, 101.3)
- moved JP5 0.09 mm to (114.9, 91.7), turned to 0 degrees
Routing:
- net AGND: track 48.7 -> 262.7 mm, vias 5 -> 18
- net GND: track 50.8 -> 149.8 mm, vias 4 -> 9
- net AVSS: track 98.8 -> 195.5 mm, vias 2 -> 16
- net AVDD: track 178.2 -> 272.1 mm, vias 8 -> 12
- net SPI_IN: track 1.47 -> 89.8 mm, vias 1 -> 4
- net -15V_Supply: track 6.58 -> 71.7 mm, vias 0 -> 1
- net 5V_Supply: track 55.9 -> 120.9 mm, vias 2 -> 10
- net SPI_CLK: track 43.6 -> 88.5 mm, vias 1 -> 2
- net VREFP: track 26.6 -> 67.3 mm
- net SPI_CS1: track 6.74 -> 30.0 mm, vias 1 -> 2
- net /RESET: track 109.3 -> 131.0 mm, vias 2 -> 4
- net DVDD: track 145.6 -> 164.5 mm, vias 10 -> 14
- net /PWDN: track 93.0 -> 111.2 mm, vias 7 -> 9
- net CLKSEL: track 53.2 -> 56.0 mm, vias 2 -> 3
- net Net-(U18-Pad43): track 58.3 -> 60.6 mm
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
Commit message: Update
Parts:
- moved C35 52.2 mm to (139.4, 115.8)
- moved C34 52.1 mm to (136.6, 115.8)
- moved TP6 52.1 mm to (174.0, 139.7)
- moved C42 52.1 mm to (182.5, 81.3)
- moved C48 52.1 mm to (184.2, 104.1)
- moved R32 52.1 mm to (178.6, 97.5)
- moved C15 52.1 mm to (132.4, 127.1)
- moved C22 52.1 mm to (158.1, 58.4)
- moved C23 52.1 mm to (117.4, 92.3)
- moved C24 52.1 mm to (110.8, 91.9)
- moved C27 52.1 mm to (145.3, 127.1)
- moved C33 52.1 mm to (147.9, 127.1)
- moved C74 52.1 mm to (118.0, 84.2)
- moved C80 52.1 mm to (111.3, 72.4)
- moved D2 52.1 mm to (122.1, 72.4)
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Routing:
- net AVSS: track 195.5 -> 214.7 mm, vias 16 -> 20
- net /PWDN: track 111.2 -> 106.8 mm
- net /RESET: track 131.0 -> 132.8 mm
- net AVDD: track 272.1 -> 273.9 mm
- net AGND: track 262.7 -> 264.3 mm, vias 18 -> 20

Commit message: Update
Changed lines of the file:
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@@
     (links 422)
     (no_connects 0)
-    (area 32.1 15.9 173.700001 127.250001)
+    (area 92.126999 54.903299 188.281301 143.066001)
     (thickness 1.6)
     (drawings 8)
@@
   (gr_line (start 188.202 142.991) (end 140.202 142.991) (angle 90) (layer Edge.Cuts) (width 0.15))
   (gr_line (start 188.202 54.991) (end 188.202 142.991) (angle 90) (layer Edge.Cuts) (width 0.15))
-  (gr_line (start 92.1809 54.9783) (end 188.1809 54.9783) (angle 90) (layer Edge.Cuts) (width 0.15))
+  (gr_line (start 92.2063 54.9783) (end 188.2063 54.9783) (angle 90) (layer Edge.Cuts) (width 0.15))
   (segment (start 165.6715 82.9945) (end 165.7004 82.9656) (width 0.25) (layer F.Cu) (net 0))
   (segment (start 155.7535 94.615) (end 155.7535 95.492) (width 0.25) (layer F.Cu) (net 1))

Commit message: Update
Routing:
- net -15V_Supply: track 71.7 -> 66.2 mm
Changed lines of the file:
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@@
     (links 422)
     (no_connects 0)
-    (area 92.126999 54.903299 188.281301 143.066001)
+    (area 73.267 48.285 189.841 144.415833)
     (thickness 1.6)
     (drawings 8)
-    (tracks 2422)
+    (tracks 2425)
     (zones 0)
     (modules 167)
@@
     (pad_to_mask_clearance 0.2)
     (aux_axis_origin 0 0)
-    (visible_elements 7FFFFF9F)
+    (visible_elements 7FFFFD9F)
     (pcbplotparams
       (layerselection 0x00030_80000001)
@@
       (padsonsilk false)
       (subtractmaskfromsilk false)
-      (outputformat 1)
+      (outputformat 4)
       (mirror false)
-      (drillshape 1)
+      (drillshape 0)
       (scaleselection 1)
-      (outputdirectory ""))
+      (outputdirectory E:/Seminar/))
   )
   (net 0 "")
@@
   (segment (start 174.604 111.012) (end 177.6555 111.012) (width 0.25) (layer F.Cu) (net 27))
   (segment (start 177.6555 111.012) (end 177.959 111.3155) (width 0.25) (layer F.Cu) (net 27))
+  (segment (start 176.11725 128.49225) (end 176.11725 130.89255) (width 0.25) (layer B.Cu) (net 28))
+  (segment (start 158.242 140.716) (end 152.7175 140.716) (width 0.25) (layer B.Cu) (net 28))
+  (segment (start 163.0045 135.9535) (end 158.242 140.716) (width 0.25) (layer B.Cu) (net 28))
+  (segment (start 171.0563 135.9535) (end 163.0045 135.9535) (width 0.25) (layer B.Cu) (net 28))
+  (segment (start 176.11725 130.89255) (end 171.0563 135.9535) (width 0.25) (layer B.Cu) (net 28))
   (via (at 174.604 106.412) (size 0.6) (drill 0.4) (layers F.Cu B.Cu) (net 28))
   (segment (start 177.9015 106.412) (end 174.604 106.412) (width 0.25) (layer F.Cu) (net 28))
-  (segment (start 152.9334 140.9319) (end 151.384 139.3825) (width 0.25) (layer B.Cu) (net 28))
-  (segment (start 175.286898 140.9319) (end 152.9334 140.9319) (width 0.25) (layer B.Cu) (net 28))
-  (segment (start 176.0855 140.133298) (end 175.286898 140.9319) (width 0.25) (layer B.Cu) (net 28))
-  (segment (start 176.0855 128.524) (end 176.0855 140.133298) (width 0.25) (layer B.Cu) (net 28))
-  (segment (start 182.3085 122.301) (end 176.0855 128.524) (width 0.25) (layer B.Cu) (net 28))
+  (segment (start 152.7175 140.716) (end 151.384 139.3825) (width 0.25) (layer B.Cu) (net 28))
+  (segment (start 182.3085 122.301) (end 176.11725 128.49225) (width 0.25) (layer B.Cu) (net 28))
+  (segment (start 176.11725 128.49225) (end 176.0855 128.524) (width 0.25) (layer B.Cu) (net 28))
   (segment (start 182.3085 114.1165) (end 182.3085 122.301) (width 0.25) (layer B.Cu) (net 28))
   (segment (start 174.604 106.412) (end 182.3085 114.1165) (width 0.25) (layer B.Cu) (net 28))

Commit message: Update
Parts:
- removed J6: DB15_F-RA, Connectors:DB15FC
- removed JP30, JP31, JP32, JP33, JP34, JP35, JP36, JP37: JP2x2, Jumper:Jumper2x2
- added C36: 1uF, Capacitors_SMD:C_1206_HandSoldering, F.Cu at (136.8, 106.8)
- added C37: 1uF, Capacitors_SMD:C_1206_HandSoldering, F.Cu at (136.8, 109.2)
- C12, C17, C18, C20, C21, C34, C35, C5, C68, C69, C76, C77, JP18, JP19, R12, R3, R4, R67, R75, R8: moved to F.Cu
- moved C69 50.3 mm to (155.3, 134.3), turned to 90 degrees
- moved C68 48.6 mm to (157.9, 134.3), turned to 90 degrees
- moved PSK3 39.3 mm to (182.0, 130.2), turned to 0 degrees
- moved R74 38.7 mm to (176.8, 140.6), turned to 0 degrees
- moved J7 37.7 mm to (111.9, 112.1), turned to 270 degrees
- moved R7 37.0 mm to (157.3, 87.3)
- moved PSK2 36.8 mm to (94.9, 66.1)
- moved R67 36.5 mm to (154.2, 70.8)
- moved C6 35.0 mm to (156.0, 113.9), turned to 270 degrees
- moved PSK5 34.1 mm to (111.9, 103.6), turned to 270 degrees
- moved R12 33.2 mm to (141.2, 118.5), turned to 180 degrees
- moved C16 30.7 mm to (158.5, 113.9), turned to 270 degrees
- moved TP8 29.4 mm to (148.6, 139.3)
- moved C4 27.0 mm to (160.9, 113.9), turned to 270 degrees
- moved C14 23.8 mm to (163.3, 113.9), turned to 270 degrees
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Connections:
- J1 pad 1: ECG_13P -> ECG_9N
- J1 pad 10: ECG_11P -> ECG_13P
- J1 pad 11: ECG_15N -> ECG_14N
- J1 pad 12: ECG_11N -> ECG_14P
- J1 pad 13: ECG_16P -> ECG_15N
- J1 pad 14: ECG_12P -> ECG_15P
- J1 pad 16: ECG_12N -> ECG_16P
- J1 pad 3: ECG_13N -> ECG_10N
- J1 pad 4: ECG_9N -> ECG_10P
- J1 pad 5: ECG_14P -> ECG_11N
- J1 pad 6: ECG_10P -> ECG_11P
- J1 pad 7: ECG_14N -> ECG_12N
- J1 pad 8: ECG_10N -> ECG_12P
- J1 pad 9: ECG_15P -> ECG_13N
- J7 pad 1: PACEOUT22 -> GPIO11
- J7 pad 10: GPIO11 -> /PWDN
- J7 pad 11: Net-(J7-Pad11) -> PACEOUT12
- J7 pad 12: GPIO12 -> PACEOUT21
- J7 pad 13: Net-(J7-Pad13) -> PACEOUT11
- J7 pad 14: GPIO13 -> PACEOUT22
- J7 pad 15: DAISY_IN -> AVSS
- J7 pad 2: PACEOUT11 -> GPIO23
- J7 pad 3: PACEOUT21 -> GPIO12
- J7 pad 4: PACEOUT12 -> GPIO22
- J7 pad 5: GPIO23 -> GPIO13
- J7 pad 6: /PWDN -> GPIO21
- J7 pad 7: GPIO22 -> Net-(J7-Pad7)
- J7 pad 8: Net-(J7-Pad8) -> DAISY_IN
- J7 pad 9: GPIO21 -> Net-(J7-Pad9)
- JP2 pad 1: Net-(J3-Pad1) -> 3.3V_Supply
- JP2 pad 2: 3.3V_Supply -> Net-(J3-Pad2)
- JP3 pad 1: Net-(J3-Pad2) -> Net-(J3-Pad1)
- PSK2 pad 1: /ADC1298_ECG_FE/ELEC_V2 -> /ADC1298_ECG_FE/ELEC_RL
- PSK2 pad 10: /ADC1298_ECG_FE/ELEC_RA -> /ADC1298_ECG_FE/ELEC_V6
- PSK2 pad 2: /ADC1298_ECG_FE/ELEC_V3 -> /ADC1298_ECG_FE/ELEC_V1
- PSK2 pad 3: /ADC1298_ECG_FE/ELEC_V4 -> /ADC1298_ECG_FE/ELEC_V5
- PSK2 pad 4: /ADC1298_ECG_FE/ELEC_V5 -> /ADC1298_ECG_FE/ELEC_V4
- PSK2 pad 5: /ADC1298_ECG_FE/ELEC_V6 -> /ADC1298_ECG_FE/ELEC_V3
- PSK2 pad 6: /ADC1298_ECG_FE/ELEC_RL -> /ADC1298_ECG_FE/ELEC_V2
- PSK2 pad 7: /ADC1298_ECG_FE/ELEC_V1 -> /ADC1298_ECG_FE/ELEC_RA
- PSK3 pad 1: 5V_Supply -> 15V_Supply
- PSK3 pad 2: 3.3V_Supply -> -15V_Supply
- PSK3 pad 3: 15V_Supply -> 5V_Supply
- PSK3 pad 4: -15V_Supply -> 3.3V_Supply
- PSK5 pad 1: ECG_5P -> ECG_5N
- PSK5 pad 10: ECG_3P -> ECG_1P
- PSK5 pad 11: ECG_7N -> ECG_2N
- PSK5 pad 12: ECG_3N -> ECG_2P
- PSK5 pad 13: ECG_8P -> ECG_3N
- PSK5 pad 14: ECG_4P -> ECG_3P
- PSK5 pad 15: ECG_8N -> ECG_4N
- PSK5 pad 16: ECG_4N -> ECG_4P
- PSK5 pad 2: ECG_1P -> ECG_5P
- PSK5 pad 3: ECG_5N -> ECG_6N
- PSK5 pad 4: ECG_1N -> ECG_6P
- PSK5 pad 5: ECG_6P -> ECG_7N
- PSK5 pad 6: ECG_2P -> ECG_7P
- PSK5 pad 7: ECG_6N -> ECG_8N
- PSK5 pad 8: ECG_2N -> ECG_8P
- PSK5 pad 9: ECG_7P -> ECG_1N
- U18 pad 1: Net-(JP30-Pad2) -> ECG_16N
- U18 pad 10: Net-(JP34-Pad4) -> ECG_12P
- U18 pad 11: Net-(JP35-Pad2) -> ECG_11N
- U18 pad 12: Net-(JP35-Pad4) -> ECG_11P
- U18 pad 13: Net-(JP36-Pad2) -> ECG_10N
- U18 pad 14: Net-(JP36-Pad4) -> ECG_10P
- U18 pad 15: Net-(JP37-Pad2) -> ECG_9N
- U18 pad 16: Net-(JP37-Pad4) -> ECG_9P
- U18 pad 2: Net-(JP30-Pad4) -> ECG_16P
- U18 pad 3: Net-(JP31-Pad2) -> ECG_15N
- U18 pad 4: Net-(JP31-Pad4) -> ECG_15P
- U18 pad 5: Net-(JP32-Pad2) -> ECG_14N
- U18 pad 6: Net-(JP32-Pad4) -> ECG_14P
- U18 pad 7: Net-(JP33-Pad2) -> ECG_13N
- U18 pad 8: Net-(JP33-Pad4) -> ECG_13P
- U18 pad 9: Net-(JP34-Pad2) -> ECG_12N
Routing:
- net AGND: track 264.3 -> 28.0 mm, vias 20 -> 6
- net AVDD: track 273.9 -> 49.0 mm, vias 12 -> 1
- net AVSS: track 214.7 -> 76.5 mm, vias 20 -> 1
- net DVDD: track 164.5 -> 40.6 mm, vias 14 -> 0
- net GND: track 149.8 -> 250.7 mm, vias 9 -> 4
- net /RESET: track 132.8 -> 66.4 mm, vias 4 -> 2
- net /ADC1298_ECG_FE/ELEC_RL: track 71.4 -> 12.9 mm
- net /ADC1298_ECG_FE/ELEC_V1: track 68.6 -> 11.2 mm
- net /ADC1298_ECG_FE/ELEC_LL: track 65.2 -> 9.34 mm, vias 2 -> 0
- net /ADC1298_ECG_FE/ELEC_LA: track 62.5 -> 11.6 mm, vias 3 -> 0
- net /ADC1298_ECG_FE/ELEC_RA: track 57.9 -> 9.07 mm
- net /ADC1298_ECG_FE/ELEC_V5: track 56.2 -> 9.93 mm
- net ECG_RL: track 56.8 -> 13.6 mm
- net /ADC1298_ECG_FE/ELEC_V4: track 50.1 -> 9.00 mm
- net /ADC1298_ECG_FE/ELEC_V6: track 51.5 -> 12.2 mm, vias 2 -> 0
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