File: Seminar_Med_Tech/Seminar_Med_Tech.kicad_pcb (KiCad board)
At the start: 2 copper layers, 96 x 88 mm, 160 parts, among them J1 CONN_02X08, J3 CONN_02X10, J5 CONN_02X10, J7 CONN_02X08, U1 OPA132, U18 ADS1298, U20 ADS1298, U4 LM317T, U5 LM317T, U6 LM337K

Commit message: Update
Parts:
- moved J7 2.80 mm to (111.8, 114.9)
- moved C32 2.03 mm to (109.0, 94.4)
- moved C93 2.02 mm to (102.4, 94.4)
- moved D10 1.88 mm to (113.1, 94.4)
- moved R25 1.88 mm to (103.0, 94.2)
- moved R26 1.88 mm to (108.2, 94.3)
- moved C23 1.70 mm to (109.2, 90.4)
- moved C24 1.69 mm to (102.7, 90.4)
- moved D4 1.62 mm to (113.3, 90.5)
- moved C72 1.62 mm to (109.1, 79.4)
- moved PSK2 1.62 mm to (95.2, 64.5)
- moved D8 1.60 mm to (113.2, 60.5)
- moved C31 1.59 mm to (109.2, 60.5)
- moved C91 1.57 mm to (102.6, 79.4)
- moved C92 1.54 mm to (102.6, 60.5)
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Routing:
- net (no net): track 0.00 -> 1307.4 mm, vias 0 -> 25
- net AGND: track 28.0 -> 99.0 mm
- net Net-(JP16-Pad2): track 54.4 -> 0.00 mm
- net PACEOUT11: track 51.2 -> 0.00 mm
- net PACEOUT12: track 50.0 -> 0.00 mm
- net AVDD: track 49.0 -> 98.5 mm, vias 1 -> 10
- net Net-(C20-Pad1): track 65.8 -> 25.8 mm, vias 2 -> 0
- net /ADC1298_ECG_FE/ELEC_SHD: track 40.5 -> 1.46 mm
- net ECG_16P: track 38.7 -> 0.00 mm
- net ECG_16N: track 36.8 -> 0.00 mm
- net ECG_15P: track 36.3 -> 0.00 mm
- net ECG_15N: track 34.6 -> 0.00 mm
- net PACEOUT22: track 34.8 -> 0.83 mm, vias 1 -> 0
- net ECG_14P: track 33.9 -> 0.00 mm
- net ECG_14N: track 32.0 -> 0.00 mm
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
Commit message: Update
Routing:
- net ECG_8N: track 50.1 -> 75.8 mm
- net ECG_8P: track 53.4 -> 76.6 mm
- net ECG_7N: track 49.6 -> 70.3 mm
- net ECG_7P: track 52.3 -> 70.7 mm
- net ECG_6P: track 60.5 -> 61.4 mm
- net ECG_5N: track 53.5 -> 54.3 mm
- net ECG_6N: track 62.4 -> 63.1 mm

Commit message: Update
Parts:
- moved TP6 14.6 mm to (162.5, 130.9)
- moved TP5 11.6 mm to (164.6, 130.8)
- moved TP3 11.1 mm to (169.3, 130.8)
- moved PSK3 10.8 mm to (173.5, 136.8), turned to 90 degrees
- moved R74 10.6 mm to (173.3, 130.6)
- moved TP4 10.00 mm to (166.9, 130.9)
- moved C68 2.36 mm to (160.0, 133.3)
- moved C69 2.36 mm to (157.4, 133.3)
- moved JP3 2.36 mm to (154.3, 132.9)
- moved TP7 2.36 mm to (160.0, 138.2)
- moved R15 2.32 mm to (145.5, 116.3), turned to 90 degrees
- moved C36 2.18 mm to (139.0, 106.8)
- moved C37 2.18 mm to (138.9, 109.0)
- moved JP1 1.53 mm to (133.5, 69.1)
- moved JP17 1.40 mm to (133.5, 60.3)
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Connections:
- J7 pad 11: PACEOUT12 -> Net-(J7-Pad11)
- J7 pad 13: PACEOUT11 -> PACEOUT12
- J7 pad 15: AVSS -> PACEOUT11
Routing:
- net (no net): track 1307.4 -> 0.00 mm, vias 25 -> 0
- net AVDD: track 98.5 -> 263.3 mm, vias 10 -> 15
- net DVDD: track 40.6 -> 164.4 mm, vias 0 -> 6
- net AGND: track 99.0 -> 201.0 mm, vias 6 -> 16
- net AVSS: track 73.3 -> 156.4 mm, vias 1 -> 11
- net PACEOUT11: track 0.00 -> 54.3 mm
- net Net-(JP16-Pad2): track 0.00 -> 53.3 mm
- net PACEOUT12: track 0.00 -> 52.8 mm
- net ECG_16P: track 0.00 -> 41.9 mm
- net Net-(C20-Pad1): track 25.8 -> 67.4 mm, vias 0 -> 2
- net ECG_16N: track 0.00 -> 40.7 mm
- net /ADC1298_ECG_FE/ELEC_SHD: track 1.46 -> 40.9 mm
- net ECG_15P: track 0.00 -> 37.5 mm
- net ECG_15N: track 0.00 -> 35.9 mm
- net ECG_14P: track 0.00 -> 34.6 mm
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
Commit message: Update
Parts:
- moved C12 16.4 mm to (143.8, 95.7)
- moved C13 16.4 mm to (126.0, 66.6)
- moved C14 16.4 mm to (147.1, 111.6)
- moved C16 16.4 mm to (142.3, 111.6)
- moved C17 16.4 mm to (142.3, 103.3)
- moved C21 16.4 mm to (140.8, 56.1)
- moved C25 16.4 mm to (118.3, 124.3)
- moved C3 16.4 mm to (123.4, 66.6)
- moved C35 16.4 mm to (120.4, 101.0)
- moved C39 16.4 mm to (157.1, 88.7)
- moved C44 16.4 mm to (158.0, 115.1)
- moved C48 16.4 mm to (154.7, 116.8)
- moved C5 16.4 mm to (143.8, 93.6)
- moved D14 16.4 mm to (149.8, 100.4)
- moved D15 16.4 mm to (149.9, 111.5)
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Other:
- outline, holes or cut-outs redrawn

Commit message: Update
Parts:
- removed C68: 100uF, Capacitors_SMD:C_1206_HandSoldering
- removed C69: 0.1uF, Capacitors_SMD:C_1206_HandSoldering
- removed C72, C73, C74, C75, C80, C82, C84, C86, C88, C91, C92, C93: 47pF, Capacitors_SMD:C_1206_HandSoldering
- removed C76, C77: 1uF, Capacitors_SMD:C_1206_HandSoldering
- removed C90: 100pF, Capacitors_SMD:C_1206_HandSoldering
- removed C95: 10uF, Capacitors_SMD:C_1206_HandSoldering
- removed D14, D15: D, Diodes_SMD:D_SOD-123
- removed J5: CONN_02X10, Pin_Headers:Pin_Header_Straight_2x10_Pitch2.54mm
- removed J7: CONN_02X08, Pin_Headers:Pin_Header_Straight_2x08_Pitch2.54mm
- removed JP21: Jumper_NC_Dual, Jumper:jumper1x3
- removed JP22, JP23, JP24, JP25, JP26, JP27, JP28, JP29: JP2x2, Jumper:Jumper2x2
- removed R43: 22.1k, Resistors_SMD:R_0805_HandSoldering
- removed R44, R67, R75: 10k, Resistors_SMD:R_0805_HandSoldering
- removed R74: 0, Resistors_SMD:R_0805_HandSoldering
- added C40: 100pF, Capacitors_SMD:C_1206_HandSoldering, F.Cu at (118.9, 54.9)
- added C41: 10uF, Capacitors_SMD:C_1206_HandSoldering, F.Cu at (120.3, 90.2)
- added C49: 100uF, Capacitors_SMD:C_1206_HandSoldering, F.Cu at (143.8, 130.9)
- added C50: 0.1uF, Capacitors_SMD:C_1206_HandSoldering, F.Cu at (140.8, 130.8)
- added C51: 47pF, Capacitors_SMD:C_1206_HandSoldering, B.Cu at (92.8, 77.1)
- added C52: 47pF, Capacitors_SMD:C_1206_HandSoldering, B.Cu at (92.9, 73.2)
- added C53: 47pF, Capacitors_SMD:C_1206_HandSoldering, B.Cu at (93.0, 80.8)
- added C54: 47pF, Capacitors_SMD:C_1206_HandSoldering, B.Cu at (92.9, 61.8)
- added C55: 1uF, Capacitors_SMD:C_1206_HandSoldering, F.Cu at (131.2, 66.6)
- added C56: 1uF, Capacitors_SMD:C_1206_HandSoldering, F.Cu at (128.7, 66.6)
- added C57: 47pF, Capacitors_SMD:C_1206_HandSoldering, B.Cu at (86.3, 73.2)
- added C58: 47pF, Capacitors_SMD:C_1206_HandSoldering, B.Cu at (86.3, 65.6)
- added C59: 47pF, Capacitors_SMD:C_1206_HandSoldering, B.Cu at (86.4, 61.8)
- added C60: 47pF, Capacitors_SMD:C_1206_HandSoldering, B.Cu at (86.5, 80.8)
- added C61: 47pF, Capacitors_SMD:C_1206_HandSoldering, B.Cu at (86.3, 84.5)
- added C63: 47pF, Capacitors_SMD:C_1206_HandSoldering, B.Cu at (86.3, 77.1)
- added C64: 47pF, Capacitors_SMD:C_1206_HandSoldering, B.Cu at (86.4, 58.2)
- added C65: 47pF, Capacitors_SMD:C_1206_HandSoldering, B.Cu at (86.3, 92.0)
- added D11: D, Diodes_SMD:D_SOD-123, F.Cu at (149.6, 89.1)
- added D12: D, Diodes_SMD:D_SOD-123, F.Cu at (149.7, 100.5)
- added J2: CONN_02X10, Pin_Headers:Pin_Header_Straight_2x10_Pitch2.54mm, F.Cu at (136.5, 80.4)
- added JP10: NI, Jumper:jumper1x3, F.Cu at (139.5, 103.3)
- added JP11: Jumper_NC_Dual, Jumper:jumper1x3, F.Cu at (136.6, 65.8)
- added JP12: JP2x2, Jumper:Jumper2x2, F.Cu at (103.3, 56.6)
- added JP13: JP2x2, Jumper:Jumper2x2, F.Cu at (103.4, 61.9)
- added JP14: JP2x2, Jumper:Jumper2x2, F.Cu at (103.4, 67.1)
- added JP6: Jumper_NC_Dual, Jumper:jumper1x3, F.Cu at (127.2, 54.6)
- added JP7: Jumper_NC_Dual, Jumper:jumper1x3, F.Cu at (111.0, 54.8)
- added JP8: NI, Jumper:jumper1x3, F.Cu at (117.3, 58.0)
- added JP9: NI, Jumper:jumper1x3, F.Cu at (127.7, 103.1)
- added PSK6: CONN_02X08, Pin_Headers:Pin_Header_Straight_2x08_Pitch2.54mm, F.Cu at (95.6, 123.9)
- added R16: 22.1k, Resistors_SMD:R_0805_HandSoldering, F.Cu at (87.0, 69.4)
- added R19: 22.1k, Resistors_SMD:R_0805_HandSoldering, F.Cu at (87.0, 65.5)
- added R23: 47, Resistors_SMD:R_0805_HandSoldering, F.Cu at (161.5, 101.4)
- added R24: 22.1k, Resistors_SMD:R_0805_HandSoldering, F.Cu at (87.1, 61.9)
- added R38: 0, Resistors_SMD:R_0805_HandSoldering, F.Cu at (158.1, 128.3)
- J1: value CONN_02X08 -> CONN_02X10; footprint Pin_Headers:Pin_Header_Straight_2x08_Pitch2.54mm -> Pin_Headers:Pin_Header_Straight_2x10_Pitch2.54mm
- J3: value CONN_02X10 -> CONN_02X08; footprint Pin_Headers:Pin_Header_Straight_2x10_Pitch2.54mm -> Pin_Headers:Pin_Header_Straight_2x08_Pitch2.54mm
- JP15, JP16: value Jumper_NC_Dual -> JP2x2; footprint Jumper:jumper1x3 -> Jumper:Jumper2x2
- JP17, JP18, JP19: value NI -> JP2x2; footprint Jumper:jumper1x3 -> Jumper:Jumper2x2
- R17, R21, R25, R29, R37, R39: value 22.1k -> 10k
- R18: value 10k -> 120
- R20: value 120 -> 22.1k
- R22: value 10k -> 270
- R26: value 10k -> 47
- R27: value 270 -> 240
- R28: value 47 -> 22.1k
- R30: value 10k -> 240
- R31: value 47 -> 10k
- R32, R35: value 240 -> 22.1k
- moved R31 88.6 mm to (92.4, 58.2), turned to 180 degrees
- moved R30 82.6 mm to (157.3, 112.5), turned to 0 degrees
- moved R32 81.9 mm to (87.0, 58.1), turned to 180 degrees
- moved R28 76.4 mm to (87.1, 84.5), turned to 180 degrees
- moved R20 74.7 mm to (87.0, 92.0), turned to 180 degrees
- moved R35 74.3 mm to (87.0, 88.1), turned to 180 degrees
- moved R26 73.0 mm to (162.1, 112.6), turned to 0 degrees
- moved R18 72.2 mm to (161.6, 90.1), turned to 0 degrees
- moved R22 69.0 mm to (156.6, 90.1), turned to 0 degrees
- moved R37 52.1 mm to (137.9, 68.4)
- moved J3 42.4 mm to (95.5, 112.6), turned to 270 degrees
- moved J1 40.8 mm to (136.5, 123.5), turned to 90 degrees
- moved R39 40.3 mm to (127.5, 77.2)
- moved JP19 37.6 mm to (103.4, 93.0), turned to 0 degrees
- moved R25 30.6 mm to (92.4, 61.8)
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Connections:
- D13 pad 1: 5V_Supply -> -15V_Supply
- D13 pad 2: DVDD -> AVSS
- J1 pad 1: ECG_9N -> Net-(J1-Pad1)
- J1 pad 10: ECG_13P -> Net-(J1-Pad10)
- J1 pad 11: ECG_14N -> Net-(J1-Pad11)
- J1 pad 12: ECG_14P -> Net-(J1-Pad12)
- J1 pad 13: ECG_15N -> SPI_CLK
- J1 pad 14: ECG_15P -> Net-(J1-Pad14)
- J1 pad 15: ECG_16N -> SPI_CS2
- J1 pad 16: ECG_16P -> Net-(J1-Pad16)
- J1 pad 2: ECG_9P -> Net-(J1-Pad2)
- J1 pad 3: ECG_10N -> Net-(J1-Pad3)
- J1 pad 4: ECG_10P -> GND
- J1 pad 5: ECG_11N -> Net-(J1-Pad5)
- J1 pad 6: ECG_11P -> Net-(J1-Pad6)
- J1 pad 7: ECG_12N -> Net-(J1-Pad7)
- J1 pad 8: ECG_12P -> Net-(J1-Pad8)
- J1 pad 9: ECG_13N -> SPI_DRDY2
- J3 pad 1: Net-(J3-Pad1) -> GPIO11
- J3 pad 10: Net-(J3-Pad10) -> /PWDN
- J3 pad 12: Net-(J3-Pad12) -> PACEOUT21
- J3 pad 13: SPI_CLK -> PACEOUT12
- J3 pad 14: Net-(J3-Pad14) -> PACEOUT22
- J3 pad 15: SPI_CS2 -> PACEOUT11
- J3 pad 16: Net-(J3-Pad16) -> AGND
- J3 pad 2: Net-(J3-Pad2) -> GPIO23
- J3 pad 3: Net-(J3-Pad3) -> GPIO12
- J3 pad 4: GND -> GPIO22
- J3 pad 5: Net-(J3-Pad5) -> GPIO13
- J3 pad 6: Net-(J3-Pad6) -> GPIO21
- J3 pad 8: Net-(J3-Pad8) -> DAISY_IN
- J3 pad 9: SPI_DRDY2 -> Net-(J3-Pad9)
- JP15 pad 1: AGND -> Net-(JP12-Pad1)
- JP15 pad 2: /ADC1298_ECG_FE/ELEC_SHD -> ECG_5N
- JP15 pad 3: ECG_SHD_DRV -> ECG_V3
- JP16 pad 1: /WCT -> Net-(JP12-Pad1)
- JP16 pad 2: Net-(JP16-Pad2) -> ECG_4N
- JP16 pad 3: AGND -> ECG_V2
- JP17 pad 1: ECG_RL -> ECG_RA
- JP17 pad 2: Net-(JP17-Pad2) -> ECG_3N
- JP17 pad 3: Net-(C20-Pad1) -> ECG_LL
- JP18 pad 1: Net-(JP18-Pad1) -> ECG_RA
- JP18 pad 2: /CLK -> ECG_2N
- JP18 pad 3: EXT_CLK -> ECG_LA
- JP19 pad 1: DVDD -> Net-(JP12-Pad1)
- JP19 pad 2: Net-(JP19-Pad2) -> ECG_1N
- JP19 pad 3: AGND -> ECG_V6
- JP2 pad 2: Net-(J3-Pad2) -> Net-(J1-Pad2)
- JP3 pad 1: Net-(J3-Pad1) -> Net-(J1-Pad1)
- OSC1 pad 1: Net-(JP19-Pad2) -> Net-(JP10-Pad2)
- OSC1 pad 3: Net-(JP18-Pad1) -> Net-(JP9-Pad1)
- PSK4 pad 2: /ADC1298_ECG_FE/ELEC_SHD -> Net-(JP6-Pad2)
- R17 pad 1: Net-(C28-Pad1) -> ECG_V4
- R17 pad 2: /ADC1298_ECG_FE/ELEC_V4 -> Net-(C28-Pad1)
- R18 pad 1: ECG_V4 -> Net-(C38-Pad1)
- R18 pad 2: Net-(C28-Pad1) -> GND
- R20 pad 1: Net-(C38-Pad1) -> Net-(C65-Pad1)
- R20 pad 2: GND -> /ADC1298_ECG_FE/ELEC_V6
- R21 pad 1: Net-(C82-Pad1) -> ECG_V6
- R21 pad 2: /ADC1298_ECG_FE/ELEC_V5 -> Net-(C65-Pad1)
- R22 pad 1: ECG_V5 -> DVDD
- R22 pad 2: Net-(C82-Pad1) -> Net-(C38-Pad1)
- R25 pad 1: Net-(C93-Pad1) -> ECG_V1
- R25 pad 2: /ADC1298_ECG_FE/ELEC_V6 -> Net-(C59-Pad1)
- R26 pad 1: ECG_V6 -> Net-(C44-Pad1)
- R26 pad 2: Net-(C93-Pad1) -> GND
- R27 pad 1: DVDD -> AVDD
- R27 pad 2: Net-(C38-Pad1) -> Net-(C43-Pad1)
- R28 pad 1: Net-(C43-Pad1) -> Net-(C61-Pad1)
- R28 pad 2: GND -> /ADC1298_ECG_FE/ELEC_LL
- R29 pad 1: Net-(C84-Pad1) -> ECG_LL
- R29 pad 2: /ADC1298_ECG_FE/ELEC_V1 -> Net-(C61-Pad1)
- R30 pad 1: ECG_V1 -> AVSS
- R30 pad 2: Net-(C84-Pad1) -> Net-(C44-Pad1)
- R31 pad 1: Net-(C44-Pad1) -> ECG_RL
- R31 pad 2: GND -> Net-(C64-Pad1)
- R32 pad 1: AVDD -> Net-(C64-Pad1)
- R32 pad 2: Net-(C43-Pad1) -> /ADC1298_ECG_FE/ELEC_RL
- R33 pad 2: /ADC1298_ECG_FE/ELEC_LL -> /ADC1298_ECG_FE/ELEC_RA
- R34 pad 1: ECG_LL -> ECG_RA
- R35 pad 1: AVSS -> Net-(C24-Pad1)
- R35 pad 2: Net-(C44-Pad1) -> /ADC1298_ECG_FE/ELEC_LA
- R36 pad 1: ECG_RL -> ECG_LA
- R36 pad 2: Net-(C92-Pad1) -> Net-(C24-Pad1)
- R37 pad 1: Net-(C92-Pad1) -> DVDD
- R37 pad 2: /ADC1298_ECG_FE/ELEC_RL -> CLKSEL
- R39 pad 1: Net-(C86-Pad1) -> DVDD
- R39 pad 2: /ADC1298_ECG_FE/ELEC_RA -> SPI_CS1
- R4 pad 2: Net-(JP17-Pad2) -> Net-(JP8-Pad2)
- R40 pad 1: ECG_RA -> ECG_V5
- R40 pad 2: Net-(C86-Pad1) -> Net-(C58-Pad1)
Routing:
- net Net-(JP12-Pad1): track 0.00 -> 53.6 mm
- net Net-(JP16-Pad2): track 53.3 -> 0.00 mm
- net Net-(JP6-Pad2): track 0.00 -> 40.9 mm
- net /ADC1298_ECG_FE/ELEC_SHD: track 40.9 -> 0.00 mm
- net Net-(J2-Pad19): track 0.00 -> 28.5 mm
- net Net-(J5-Pad19): track 28.5 -> 0.00 mm
- net Net-(J3-Pad2): track 14.6 -> 0.00 mm
- net Net-(J1-Pad2): track 0.00 -> 14.6 mm
- net Net-(J3-Pad1): track 6.33 -> 0.00 mm
- net Net-(J1-Pad1): track 0.00 -> 6.33 mm
- net Net-(JP8-Pad2): track 0.00 -> 6.18 mm
- net Net-(JP17-Pad2): track 6.18 -> 0.00 mm
- net Net-(JP19-Pad2): track 5.05 -> 0.00 mm
- net Net-(JP10-Pad2): track 0.00 -> 5.05 mm
- net Net-(JP9-Pad1): track 0.00 -> 4.05 mm
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