File: Seminar_Med_Tech/_autosave-Seminar_Med_Tech.kicad_pcb (KiCad board)
At the start: 2 copper layers, 98.6 x 88 mm, 167 parts, among them J1 CONN_02X08, J3 CONN_02X10, J5 CONN_02X10, J6 DB15_F-RA, J7 CONN_02X08, U1 OPA132, U18 ADS1298, U20 ADS1298, U4 LM317T, U5 LM317T, U6 LM337K

Commit message: Update
Parts:
- C23, C24, C26, C28, C29, C30, C31, C32, C72, C73, C74, C75, C80, C82, C84, C86, C88, C91, C92, C93: moved to F.Cu
- JP16: value Jumper_NC_Dual -> Jumper
- moved C43 88.0 mm to (135.6, 41.8)
- moved D14 88.0 mm to (134.5, 36.0)
- moved R32 88.0 mm to (134.2, 33.1)
- moved C4 55.8 mm to (133.0, 107.9)
- moved JP18 55.8 mm to (135.1, 89.3)
- moved OSC1 55.8 mm to (133.4, 71.8)
- moved C12 55.8 mm to (133.1, 105.2)
- moved C16 55.8 mm to (133.1, 94.8)
- moved C18 55.8 mm to (133.1, 102.4)
- moved C5 55.8 mm to (133.2, 97.4)
- moved JP19 55.8 mm to (135.2, 80.8)
- moved PSK3 55.3 mm to (130.7, 79.2), turned to 0 degrees
- moved J7 53.8 mm to (55.3, 89.7), turned to 180 degrees
- moved R10 48.6 mm to (67.6, 95.6)
- moved R9 48.4 mm to (57.1, 94.2), turned to 90 degrees
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Connections:
- C90 pad 2: /WCT -> Net-(C90-Pad2)
- J1 pad 10: ECG_11P -> ECG_10N
- J1 pad 12: ECG_11N -> ECG_10P
- J1 pad 14: ECG_12P -> ECG_9N
- J1 pad 16: ECG_12N -> ECG_9P
- J1 pad 2: ECG_9P -> ECG_12N
- J1 pad 4: ECG_9N -> ECG_12P
- J1 pad 6: ECG_10P -> ECG_11N
- J1 pad 8: ECG_10N -> ECG_11P
- JP16 pad 2: Net-(JP16-Pad2) -> Net-(C90-Pad2)
- JP22 pad 1: Net-(JP16-Pad2) -> /WCT
- JP23 pad 1: Net-(JP16-Pad2) -> /WCT
- JP24 pad 1: Net-(JP16-Pad2) -> /WCT
- JP25 pad 1: Net-(JP16-Pad2) -> /WCT
- JP26 pad 1: Net-(JP16-Pad2) -> /WCT
- JP29 pad 1: Net-(JP16-Pad2) -> /WCT
- PSK2 pad 10: /ADC1298_ECG_FE/ELEC_RA -> /ADC1298_ECG_FE/ELEC_RL
- PSK2 pad 6: /ADC1298_ECG_FE/ELEC_RL -> /ADC1298_ECG_FE/ELEC_RA
- PSK2 pad 7: /ADC1298_ECG_FE/ELEC_V1 -> /ADC1298_ECG_FE/ELEC_LA
- PSK2 pad 9: /ADC1298_ECG_FE/ELEC_LA -> /ADC1298_ECG_FE/ELEC_V1
- PSK5 pad 10: ECG_3P -> ECG_2N
- PSK5 pad 12: ECG_3N -> ECG_2P
- PSK5 pad 14: ECG_4P -> ECG_1N
- PSK5 pad 16: ECG_4N -> ECG_1P
- PSK5 pad 2: ECG_1P -> ECG_4N
- PSK5 pad 4: ECG_1N -> ECG_4P
- PSK5 pad 6: ECG_2P -> ECG_3N
- PSK5 pad 8: ECG_2N -> ECG_3P
- U20 pad 64: /WCT -> Net-(C90-Pad2)
Routing:
- net /ADC1298_ECG_FE/ELEC_RL: track 71.4 -> 0.00 mm
- net /ADC1298_ECG_FE/ELEC_V1: track 68.6 -> 0.00 mm
- net /ADC1298_ECG_FE/ELEC_LL: track 65.2 -> 0.00 mm, vias 2 -> 0
- net /ADC1298_ECG_FE/ELEC_LA: track 62.5 -> 0.00 mm, vias 3 -> 0
- net /ADC1298_ECG_FE/ELEC_RA: track 57.9 -> 0.00 mm
- net ECG_16N: track 57.8 -> 0.00 mm
- net /ADC1298_ECG_FE/ELEC_V5: track 56.2 -> 0.00 mm
- net /ADC1298_ECG_FE/ELEC_V6: track 51.5 -> 0.00 mm, vias 2 -> 0
- net ECG_16P: track 51.2 -> 0.00 mm
- net /ADC1298_ECG_FE/ELEC_V4: track 50.1 -> 0.00 mm
- net ECG_V6: track 47.9 -> 0.00 mm, vias 1 -> 0
- net ECG_15N: track 44.7 -> 0.00 mm
- net /ADC1298_ECG_FE/ELEC_V3: track 44.2 -> 0.00 mm
- net ECG_15P: track 37.5 -> 0.00 mm
- net ECG_4P: track 36.2 -> 0.00 mm
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Other:
- board size 98.6 x 88 mm -> 96 x 88 mm
