File: Seminar_Med_Tech/ADC1298_ECG_FE.sch (KiCad schematic (older format))
At the start: 54 parts, among them J6 DB15_F-RA

Commit message: Update
Parts:
- removed J6: DB15_F-RA, Connectors:DB15FC, symbol CONN_01X15
- renumbered C72 to C51, C73 to C52, C74 to C53, C75 to C54, C80 to C57, C82 to C58, C84 to C59, C86 to C60, C88 to C61, C91 to C63, C92 to C64, C93 to C65, JP15 to JP6, R17 to R16, R18 to R17, R21 to R19, R25 to R20, R26 to R21, R29 to R24, R30 to R25, R33 to R28, R34 to R29, R36 to R31, R37 to R32, R39 to R33, R40 to R34, R43 to R35, R44 to R36, R22 to R40
Connections:
- net ELEC_SHD: no longer names the net of JP6.2, PSK4.2 (P2)
- no-connect marks 5 -> 1
