File: Seminar_Med_Tech/Kicad/Seminar_Med_Tech.kicad_pcb (KiCad board)
At the start: 2 copper layers, 101 x 95.3 mm, 164 parts, among them J1 CONN_02X10, J2 CONN_02X10, J3 CONN_02X08, U1 OPA132, U18 ADS1298, U20 ADS1298, U4 LM317T, U5 LM317T, U6 LM337K

Commit message: Update
Parts:
- moved JP2 6.69 mm to (131.9, 123.6), turned to 0 degrees
- moved C33 0.35 mm to (135.3, 131.5)
- moved C27 0.30 mm to (132.4, 131.6)
Connections:
- JP2 pad 2: Net-(J1-Pad2) -> Net-(J1-Pad1)
- JP3 pad 1: Net-(J1-Pad1) -> Net-(J1-Pad2)
Routing:
- net GND: track 243.0 -> 230.2 mm
- net Net-(J1-Pad2): track 12.3 -> 16.9 mm
- net Net-(J1-Pad1): track 6.33 -> 3.60 mm
- net 3.3V_Supply: track 46.6 -> 45.4 mm
